File: kicad-dtm-enclosure.kicad_sch (KiCad schematic)
At the start: 1 part, among them J1 DTM13-12Px-R008

Commit message: fix footprint reference
Parts:
- J1: footprint lib_fp:DTM13-12Px-R008 -> kicad-dtm-enclosure:DTM13-12Px-R008
Changed lines of the file:
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@@
       (effects (font (size 1.524 1.524)) (justify left))
     )
-    (property "Footprint" "lib_fp:DTM13-12Px-R008" (id 2) (at 257.81 89.154 0)
+    (property "Footprint" "kicad-dtm-enclosure:DTM13-12Px-R008" (id 2) (at 257.81 89.154 0)
       (effects (font (size 1.524 1.524)) hide)
     )
@@
   (symbol_instances
     (path "/c423a343-2ddb-4623-bb67-fea63e504aa6"
-      (reference "J1") (unit 1) (value "DTM13-12Px-R008") (footprint "lib_fp:DTM13-12Px-R008")
+      (reference "J1") (unit 1) (value "DTM13-12Px-R008") (footprint "kicad-dtm-enclosure:DTM13-12Px-R008")
     )
   )
